File: CW312T-AURIX-TC233.kicad_pcb (KiCad board)
At the start: 2 copper layers, 58.7 x 53.7 mm, 24 parts, among them P1 PCIEx4 EDGE CONNECTOR, U1 TC233LP32F200NACKXUMA1, U2 LD1117SC-R

Commit message: first draft - ready for review
Parts:
- added PCB1: CE Symbol, Silkscrren_Symbols:CE-Logo_8.5x6mm_SilkScreen, F.Cu at (119.7, 107.3)
- added PCB2: Pb_Free Symbol, Silkscrren_Symbols:Pb_Free_8.0x8.0mm_SilkScreen, F.Cu at (128.6, 107.4)
- added PCB3: UKCA symbol, Silkscrren_Symbols:UKCA-Logo_8x8mm_SilkScreen, F.Cu at (138.0, 107.0)
- added PCB4: WEEE SYMBOL, Silkscrren_Symbols:WEEE-Logo_5.6x8mm_SilkScreen, F.Cu at (110.3, 106.9)
- moved R8 26.1 mm to (117.0, 82.3)
- moved R4 23.5 mm to (125.5, 82.0)
- moved C5 23.5 mm to (124.8, 76.8)
- moved C6 23.5 mm to (124.8, 78.6)
- moved C4 8.54 mm to (149.2, 93.4)
- moved C1 8.54 mm to (140.3, 100.0)
- moved C2 8.54 mm to (142.2, 100.0)
- moved C3 8.54 mm to (149.2, 91.5)
- moved R1 8.54 mm to (149.2, 95.3)
- moved R2 8.54 mm to (153.5, 100.1)
- moved U2 8.54 mm to (147.9, 102.3)
- moved R3 4.27 mm to (114.0, 102.8), turned to 180 degrees
- moved R9 4.02 mm to (114.8, 82.3), turned to -90 degrees
- moved R6 3.34 mm to (133.1, 83.4), turned to 0 degrees
- moved R7 3.17 mm to (125.0, 103.7)
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Routing:
- net +3V3: track 0.00 -> 155.0 mm, vias 0 -> 10
- net /FILT_HP: track 0.00 -> 81.7 mm, vias 0 -> 4
- net /VCORE: track 0.00 -> 74.3 mm, vias 0 -> 4
- net /RST: track 0.00 -> 66.4 mm, vias 0 -> 2
- net /CLKIN: track 0.00 -> 46.6 mm, vias 0 -> 2
- net GND: track 0.00 -> 43.6 mm, vias 0 -> 18
- net /TRST: track 0.00 -> 39.1 mm, vias 0 -> 3
- net /TX: track 0.00 -> 39.0 mm
- net /RX: track 0.00 -> 38.1 mm
- net +1V5: track 0.00 -> 38.0 mm
- net /TDO: track 0.00 -> 37.5 mm, vias 0 -> 2
- net /TDI: track 0.00 -> 36.2 mm, vias 0 -> 4
- net /GPIO3: track 0.00 -> 36.0 mm
- net /TCK: track 0.00 -> 35.2 mm, vias 0 -> 2
- net /GPIO4: track 0.00 -> 34.8 mm
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- added copper zone on B.Cu, net GND
Other:
- board text added: "AURIX Target Board For CW312T Board"
- board text added: "CW312T-AURIX NewAE Technology Inc. RoHS / Pb Free"
- board text added: "Issues wth gnd connection unsure why"

Commit message: updated schematic, pcb and production files - ready for review
Routing:
- net GND: track 43.6 -> 58.9 mm, vias 18 -> 19
- net /HWCFG5: track 25.0 -> 26.9 mm
- net /HWCFG4: track 27.4 -> 29.1 mm
- net +3V3: track 155.0 -> 155.8 mm
Other:
- board text added: "RST"
- board text added: "VREF"
- board text removed: "Issues wth gnd connection unsure why"

Commit message: updated silkscreen and production files
Routing:
- net /FILT_HP: track 81.7 -> 82.3 mm
Other:
- board text added: "+1V5"
- board text added: "+3V3"
- board text removed: "VREF"
